File: PCB/common/left.kicad_sch (KiCad schematic)
At the start: 35 parts, among them J2 TRS

Commit message: Initial left side components
Parts:
- removed U?: TPD4E05U06DQAR, Package_SON:USON-10_2.5x1.0mm_P0.5mm, symbol Power_Protection:TPD4EUSB30
- added C1, C6: 10uF, Capacitor_Tantalum_SMD:CP_EIA-2012-12_Kemet-R, symbol Device:C_Polarized_Small
- added C10, C11, C2: 4.7u, Capacitor_SMD:C_0603_1608Metric, symbol Device:C_Small
- added C12, C13: 12p, Capacitor_SMD:C_0603_1608Metric, symbol Device:C_Small
- added C9: 1u, Capacitor_SMD:C_0603_1608Metric, symbol Device:C_Small
- added D2: LED_Dual_AKKA, symbol Device:LED_Dual_AKKA
- added D24: Schottky, Diode_SMD:D_SOD-323, symbol Device:D_Schottky_Small
- added H10, H11, H12, H13: qw-logo, qw-logo:qw new logo silk + copper sm, symbol Mechanical:MountingHole
- added H14, H15, H16, H17: 1999-logo, 1999:1999 logo md, symbol Mechanical:MountingHole
- added J3: TC2030_SWD, PCM_marbastlib-various:CON_TC2030_outlined, symbol PCM_marbastlib-various:TC2030_SWD
- added J4: Battery, Connector_Molex:Molex_Pico-EZmate_78171-0002_1x02-1MP_P1.20mm_Vertical, symbol Connector_Generic_MountingPin:Conn_01x02_MountingPin
- added L2: 10 uH, Inductor_SMD:L_0603_1608Metric, symbol Device:L_Small
- added LED1: CHARGE, LED_SMD:LED_0805_2012Metric, symbol Device:LED_Small
- added Q1: AO3401A, Package_TO_SOT_SMD:SOT-23, symbol Transistor_FET:AO3401A
- added R1, R3: 5k, Resistor_SMD:R_0603_1608Metric, symbol Device:R_Small
- added R2: 10k, Resistor_SMD:R_0603_1608Metric, symbol Device:R_Small
- added R4: 806, Resistor_SMD:R_0603_1608Metric, symbol Device:R_Small
- added R5: 2M, Resistor_SMD:R_0603_1608Metric, symbol Device:R_Small
- added SW22: SW_SPDT, Button_Switch_SMD:SW_SPDT_PCM12, symbol Switch:SW_SPDT
- added SW23: SW_Push, Button_Switch_SMD:SW_SPST_SKQG_WithStem, symbol Switch:SW_Push
- added U2: nRF52840_E73-2G4M08S1C, PCM_marbastlib-various:nRF52840_E73-2G4M08S1C, symbol PCM_marbastlib-various:nRF52840_E73-2G4M08S1C
- added U3: TP4056, qw-footprints:CustomTP4056, symbol PCM_marbastlib-various:TP4056
- added U3: USBLC6-2SC6, Package_TO_SOT_SMD:SOT-23-6, symbol Power_Protection:USBLC6-2SC6
- added Y1: 32.768 KHz, Crystal:Crystal_SMD_2012-2Pin_2.0x1.2mm, symbol Device:Crystal_Small
Connections:
- net +5V: now also C1.1, C10.1, C2.1, D24.2 (A), LED1.2 (A), Q1.1 (G), R1.1, U2.27 (VBUS), U3.4 (VCC), U3.5 (VBUS), U3.8 (CE)
- net D+: now also U2.31 (D+), U3.4 (I/O2); no longer J?.A6 (D+), J?.B6 (D+)
- net D-: now also U2.29 (D-), U3.3 (I/O2); no longer J?.A7 (D-), J?.B7 (D-)
- net GND: now also C1.2, C10.2, C11.2, C12.2, C13.2, C2.2, C6.2, C9.2, J3.5 (GND), J4.1 (Pin_1), J4.MP (MountPin), R1.2, R3.2, R5.2, U2.21 (GND), U2.24 (GND), U2.5 (GND), U3.1 (TEMP), U3.2 (GND), U3.3 (GND)
- new net: C12.1, U2.11 (P0.00/XL1), Y1.2
- new net: C13.1, U2.13 (P0.01/XL2), Y1.1
- new net: R3.1, U3.2 (PROG)
- new net: R2.2, U3.7 (CHRG)
- new net: LED1.1 (K), R2.1
- new net +BATT: C6.1, J4.2 (Pin_2), R4.1, U3.5 (BAT)
- new net +VSW: C11.1, D24.1 (K), Q1.2 (S), U2.23 (VDDH)
- new net 0.02: U2.7 (P0.02/AIN0)
- new net 0.03: U2.3 (P0.03/AIN1)
- new net 0.04: U2.18 (P0.04/AIN2)
- new net 0.06: U2.14 (P0.06)
- new net 0.07: U2.22 (P0.07)
- new net 0.08: U2.16 (P0.08)
- new net 0.09: U2.41 (P0.09/NFC1)
- new net 0.10: U2.43 (P0.10/NFC2)
- new net 0.12: U2.20 (P0.12)
- new net 0.13: U2.33 (P0.13)
- new net 0.15: U2.28 (P0.15)
- new net 0.17: U2.30 (P0.17)
- new net 0.20: U2.32 (P0.20)
- new net 0.22: U2.34 (P0.22)
- new net 0.24: U2.35 (P0.24)
- new net 0.26: U2.12 (P0.26)
- new net 0.28: U2.4 (P0.28/AIN4)
- new net 0.29: U2.8 (P0.29/AIN5)
- new net 0.30: U2.10 (P0.30/AIN6)
- new net 0.31: U2.9 (P0.31/AIN7)
- new net 1.00: U2.36 (P1.00)
- new net 1.02: U2.38 (P1.02)
- new net 1.04: U2.40 (P1.04)
- new net 1.06: U2.42 (P1.06)
- new net 1.09: U2.17 (P1.09)
- new net 1.10: U2.2 (P1.10)
- new net 1.11: U2.1 (P1.11)
- new net 1.13: U2.6 (P1.13)
- new net BATTTON: Q1.3 (D)
- new net DBUS+: J?.A6 (D+), J?.B6 (D+), U3.6 (I/O1)
- new net DBUS-: J?.A7 (D-), J?.B7 (D-), U3.1 (I/O1)
- new net DCCH: L2.1, U2.25 (DCCH)
- new net RESET: J3.3 (~{RST}), U2.26 (P0.18/~{RESET})
- new net SWDCLK: J3.4 (SWCLK), U2.39 (SWDCLK)
- new net SWDIO: J3.2 (SWDIO), U2.37 (SWDIO)
- new net VDD: C9.1, J3.1 (VCC), L2.2, U2.19 (VDD)
- new net VSENSE: R4.2, R5.1, U2.15 (P0.05/AIN3)
- no-connect marks 2 -> 4
Other:
- note added: "Programming header"
- note removed: "USB ESD"
- moved on the sheet: EXSW?, SW?
